File: 2018-fri3d-workshop.kicad_pcb (KiCad board)
At the start: 2 copper layers, 50 x 60 mm, 31 parts, among them J1 USB_B, J2 Conn_01x02, J3 Conn_01x03_m, J4 Conn_01x03_m, J5 Conn_01x02, J6 GS2, J7 Conn_01x04, Q1 DMG1012UW, SW1 SW_SPST, SW2 SW_SPST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

Commit message: added designer/descripion to silkscreen
Other:
- board text added: "AV"
- board text added: "BOT"
- board text added: "Designed by: Alexander"
- board text added: "Simon Says fri3d workshop 07-2018"
- board text added: "TOP"
Changed lines of the file:
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@@
     (links 76)
     (no_connects 0)
-    (area 154.024999 59.324999 210.075001 126.305001)
+    (area 153.975099 59.325099 210.075001 126.304901)
     (thickness 1.6)
-    (drawings 15)
+    (drawings 20)
     (tracks 329)
     (zones 0)
@@
   )
   (setup
-    (last_trace_width 1)
+    (last_trace_width 0.15)
     (user_trace_width 0.25)
     (user_trace_width 0.3)
@@
       (net 2 GND))
   )
+  (gr_text AV (at 185 104) (layer F.Cu)
+    (effects (font (size 1 1) (thickness 0.15)))
+  )
+  (gr_text "Designed by:\nAlexander" (at 208 90 90) (layer F.SilkS)
+    (effects (font (size 0.9 0.9) (thickness 0.15)))
+  )
+  (gr_text "Simon Says\nfri3d workshop\n07-2018" (at 161.9 80.5) (layer F.SilkS)
+    (effects (font (size 1.5 1.5) (thickness 0.3)) (justify left))
+  )
+  (gr_text BOT (at 167 105.8) (layer B.Cu)
+    (effects (font (size 1 1) (thickness 0.15)))
+  )
+  (gr_text TOP (at 167 104.5) (layer F.Cu)
+    (effects (font (size 1 1) (thickness 0.15)))
+  )
   (gr_text GND (at 192 95 90) (layer F.SilkS)
     (effects (font (size 1 1) (thickness 0.15)))
@@
     (effects (font (size 1 1) (thickness 0.15)))
   )
-  (gr_text SWIO (at 196.5 96 360) (layer F.SilkS)
+  (gr_text SWIO (at 196.5 96) (layer F.SilkS)
     (effects (font (size 1 1) (thickness 0.15)))
   )
-  (gr_text 3v3 (at 200 96 360) (layer F.SilkS)
+  (gr_text 3v3 (at 200 96) (layer F.SilkS)
     (effects (font (size 1 1) (thickness 0.15)))
   )
@@
   (segment (start 194.180746 109.9) (end 196.1 109.9) (width 0.5) (layer F.Cu) (net 11))
   (segment (start 196.1 109.9) (end 197.222183 108.777817) (width 0.5) (layer F.Cu) (net 11))
+  (segment (start 182.05 104.325) (end 175.325 104.325) (width 0.5) (layer F.Cu) (net 12))
+  (segment (start 173.5 99.2) (end 170.7 96.4) (width 0.5) (layer F.Cu) (net 12))
+  (segment (start 163.1 80.9) (end 163.1 80.899986) (width 0.5) (layer F.Cu) (net 12))
+  (segment (start 175.325 104.325) (end 173.5 102.5) (width 0.5) (layer F.Cu) (net 12))
+  (segment (start 173.5 102.5) (end 173.5 99.2) (width 0.5) (layer F.Cu) (net 12))
+  (segment (start 170.7 96.4) (end 164.2 96.4) (width 0.5) (layer F.Cu) (net 12))
+  (segment (start 164.2 96.4) (end 162.800001 95.000001) (width 0.5) (layer F.Cu) (net 12))
+  (segment (start 162.800001 95.000001) (end 162.8 81.2) (width 0.5) (layer F.Cu) (net 12))
+  (segment (start 162.8 81.2) (end 163.1 80.9) (width 0.5) (layer F.Cu) (net 12))
   (segment (start 164.899986 79.1) (end 164.899992 79.1) (width 0.5) (layer B.Cu) (net 12))
   (segment (start 163.1 80.899986) (end 164.899986 79.1) (width 0.5) (layer B.Cu) (net 12))
@@
   (segment (start 171.222183 72.777817) (end 164.9 79.1) (width 0.5) (layer F.Cu) (net 12))
   (via (at 164.899992 79.1) (size 0.8) (drill 0.4) (layers F.Cu B.Cu) (net 12))
-  (segment (start 182.05 104.325) (end 175.325 104.325) (width 0.5) (layer F.Cu) (net 12))
-  (segment (start 175.325 104.325) (end 174.8 103.8) (width 0.5) (layer F.Cu) (net 12))
-  (segment (start 174.8 103.8) (end 174.8 100.5) (width 0.5) (layer F.Cu) (net 12))
-  (segment (start 174.8 100.5) (end 170.7 96.4) (width 0.5) (layer F.Cu) (net 12))
-  (segment (start 170.7 96.4) (end 164.2 96.4) (width 0.5) (layer F.Cu) (net 12))
-  (segment (start 164.2 96.4) (end 162.800001 95.000001) (width 0.5) (layer F.Cu) (net 12))
-  (segment (start 162.800001 95.000001) (end 162.8 81.2) (width 0.5) (layer F.Cu) (net 12))
-  (segment (start 162.8 81.2) (end 163.1 80.9) (width 0.5) (layer F.Cu) (net 12))
-  (segment (start 163.1 80.9) (end 163.1 80.899986) (width 0.5) (layer F.Cu) (net 12))
   (via (at 163.1 80.899986) (size 0.8) (drill 0.4) (layers F.Cu B.Cu) (net 12))
   (segment (start 182.05 105.625) (end 180.575 105.625) (width 0.5) (layer F.Cu) (net 13))
@@
       )
     )
+  )
+  (zone (net 0) (net_name "") (layer B.Cu) (hatch edge 0.508)
+    (connect_pads (clearance 0.3))
+    (min_thickness 0.254)
+    (keepout (tracks not_allowed) (vias not_allowed) (copperpour not_allowed))
+    (fill yes (arc_segments 16) (thermal_gap 0.508) (thermal_bridge_width 0.508))
+    (polygon
+      (pts
+        (xy 165.3 106.6) (xy 168.7 106.6) (xy 168.7 103.6) (xy 165.3 103.6)
+      )
+    )
+  )
+  (zone (net 0) (net_name "") (layer F.Cu) (hatch edge 0.508)
+    (connect_pads (clearance 0.3))
+    (min_thickness 0.254)
+    (keepout (tracks not_allowed) (vias not_allowed) (copperpour not_allowed))
+    (fill yes (arc_segments 16) (thermal_gap 0.508) (thermal_bridge_width 0.508))
+    (polygon
+      (pts
+        (xy 165.3 103.6) (xy 168.7 103.6) (xy 168.7 106.6) (xy 165.3 106.6)
+      )
+    )

Commit message: Fixed EN and GND pin regulator
Connections:
- U1 pad 2: Vusb -> GND
- U1 pad 3: GND -> Vusb
Routing:
- net Vusb: track 59.0 -> 62.2 mm, vias 0 -> 2
- net GND: track 248.4 -> 248.2 mm, vias 17 -> 18
Other:
- outline, holes or cut-outs redrawn
- rule pad_to_mask_clearance: 0.15 -> 0
- board text added: "Designed by: Alexander 07-2018"
- board text added: "Simon Says fri3d workshop"
- board text removed: "Designed by: Alexander"
- board text removed: "Simon Says fri3d workshop 07-2018"
